Commit message: delete duplication

File: stella_description/urdf/stella_navi.urdf.xacro (robot description, xacro)
@@ -216,194 +216,3 @@
   </joint>
   <link name="cam_link"/>
-  <gazebo reference="base_link">
-    <material>Gazebo/DarkGrey</material>
-  </gazebo>
-  <gazebo reference="imu_link">
-    <gravity>true</gravity>
-    <sensor type="imu" name="imu">
-      <always_on>true</always_on>
-      <update_rate>100</update_rate>
-      <imu>
-        <angular_velocity>
-          <x>
-            <noise type="gaussian">
-              <mean>0.0</mean>
-              <stddev>2e-4</stddev>
-            </noise>
-          </x>
-          <y>
-            <noise type="gaussian">
-              <mean>0.0</mean>
-              <stddev>2e-4</stddev>
-            </noise>
-          </y>
-          <z>
-            <noise type="gaussian">
-              <mean>0.0</mean>
-              <stddev>2e-4</stddev>
-            </noise>
-          </z>
-        </angular_velocity>
-        <linear_acceleration>
-          <x>
-            <noise type="gaussian">
-              <mean>0.0</mean>
-              <stddev>1.7e-2</stddev>
-            </noise>
-          </x>
-          <y>
-            <noise type="gaussian">
-              <mean>0.0</mean>
-              <stddev>1.7e-2</stddev>
-            </noise>
-          </y>
-          <z>
-            <noise type="gaussian">
-              <mean>0.0</mean>
-              <stddev>1.7e-2</stddev>
-            </noise>
-          </z>
-        </linear_acceleration>
-      </imu>
-      <plugin name="AHRS" filename="libgazebo_ros_imu_sensor.so">
-        <ros>
-          <namespace>imu</namespace>
-          <remapping>~/out:=data</remapping>
-        </ros>
-        <initial_orientation_as_reference>false</initial_orientation_as_reference>
-      </plugin>
-    </sensor>
-  </gazebo>
-  <gazebo reference="cam_link">
-    <sensor name="cam" type="camera">
-      <update_rate>10</update_rate>
-      <always_on>1</always_on>
-      <camera name="camera">
-        <horizontal_fov>1.3962634</horizontal_fov>
-        <image>
-          <width>1920</width>
-          <height>1080</height>
-          <format>R8G8B8</format>
-        </image>
-        <clip>
-          <near>0.01</near>
-          <far>20</far>
-        </clip>
-        <distortion>
-          <k1>0.0</k1>
-          <k2>0.0</k2>
-          <k3>0.0</k3>
-          <p1>0.0</p1>
-          <p2>0.0</p2>
-          <center>0.5 0.5</center>
-        </distortion>
-      </camera>
-      <plugin filename="libgazebo_ros_camera.so" name="cam_controller">
-        <ros>
-          <remapping>~/image_raw:=image_raw</remapping>
-          <remapping>~/camera_info:=camera_info</remapping>
-        </ros>
-        <camera_name>camera</camera_name>
-        <frame_name>cam_link</frame_name>
-      </plugin>
-    </sensor>
-  </gazebo>
-  <gazebo reference="base_scan">
-    <material>Gazebo/FlatBlack</material>
-    <sensor type="ray" name="ydlidar">
-      <pose>0 0 0 0 0 0</pose>
-      <ray>
-        <scan>
-          <horizontal>
-            <samples>360</samples>
-            <resolution>2.0</resolution>
-            <min_angle>-3.141592</min_angle>
-            <max_angle>3.141592</max_angle>
-          </horizontal>
-        </scan>
-        <range>
-          <min>0.12</min>
-          <max>10.0</max>
-          <resolution>0.015</resolution>
-        </range>
-        <noise>
-          <type>gaussian</type>
-          <mean>0.0</mean>
-          <stddev>0.01</stddev>
-        </noise>
-      </ray>
-      <always_on>true</always_on>
-      <visualize>false</visualize>
-      <update_rate>5</update_rate>
-      <plugin name="ydlidar" filename="libgazebo_ros_ray_sensor.so">
-        <ros>
-          <remapping>~/out:=scan</remapping>
-        </ros>
-        <output_type>sensor_msgs/LaserScan</output_type>
-      </plugin>
-    </sensor>
-  </gazebo>
-  <gazebo reference="caster_link">
-    <kp>500000.0</kp>
-    <kd>50.0</kd>
-    <mu1>0.1</mu1>
-    <mu2>0.1</mu2>
-    <material>Gazebo/FlatBlack</material>
-  </gazebo>
-  <gazebo reference="caster_wheel_link">
-    <kp>500000.0</kp>
-    <kd>50.0</kd>
-    <mu1>0.1</mu1>
-    <mu2>0.1</mu2>
-    <material>Gazebo/FlatBlack</material>
-  </gazebo>
-  <gazebo reference="wheel_l_link">
-    <kp>500000.0</kp>
-    <kd>50.0</kd>
-    <mu1>5.0</mu1>
-    <mu2>5.0</mu2>
-    <material>Gazebo/FlatBlack</material>
-  </gazebo>
-  <gazebo reference="wheel_r_link">
-    <kp>500000.0</kp>
-    <kd>50.0</kd>
-    <mu1>5.0</mu1>
-    <mu2>5.0</mu2>
-    <material>Gazebo/FlatBlack</material>
-  </gazebo>
-  <!-- joint publisher -->
-  <gazebo>
-    <plugin name="stella_joint_state" filename="libgazebo_ros_joint_state_publisher.so">
-      <ros>
-        <remapping>~/out:=joint_states</remapping>
-      </ros>
-      <update_rate>30</update_rate>
-      <joint_name>caster_joint</joint_name>
-      <joint_name>caster_wheel_joint</joint_name>
-      <joint_name>wheel_l_joint</joint_name>
-      <joint_name>wheel_r_joint</joint_name>
-    </plugin>
-  </gazebo>
-  <!-- differential drive -->
-  <gazebo>
-    <plugin name="stella_joint_controller" filename="libgazebo_ros_diff_drive.so">
-      <update_rate>30</update_rate>
-      <!-- wheel -->
-      <left_joint>wheel_l_joint</left_joint>
-      <right_joint>wheel_r_joint</right_joint>
-      <!-- kinematics -->
-      <wheel_separation>0.337</wheel_separation>
-      <wheel_diameter>0.18</wheel_diameter>
-      <!-- limits -->
-      <max_wheel_torque>13.5</max_wheel_torque>
-      <max_wheel_acceleration>10.43</max_wheel_acceleration>
-      <!-- output -->
-      <publish_odom>false</publish_odom>
-      <publish_odom_tf>false</publish_odom_tf>
-      <publish_wheel_tf>false</publish_wheel_tf>
-      <odometry_frame>odom</odometry_frame>
-      <odometry_topic>odom</odometry_topic>
-      <robot_base_frame>base_footprint</robot_base_frame>
-    </plugin>
-  </gazebo>
 </robot>
